File: testing 5/testing5.kicad_pcb (KiCad board)
At the start: 2 copper layers, 132 x 130 mm, 37 parts, among them J1 ESP32_GPIO, J2 Screw_Terminal_01x03, J3 Screw_Terminal_01x03, J4 Screw_Terminal_01x03, J5 Screw_Terminal_01x03, K1 SRD-05VDC-SL-C, K2 SRD-05VDC-SL-C, K3 SRD-05VDC-SL-C, K4 SRD-05VDC-SL-C, SW1 RESET, SW2 BOOT, U1 ULN2003A, U2 PC817, U3 PC817, U4 PC817, U5 PC817, U6 ESP32-S3-WROOM-1, U7 HLK-PM01, U8 AMS1117-3.3

Commit message: testing 5: merge relay+ESP32+PSU, fix PCB DRC errors 9 -> 1
Routing:
- net GND: track 259.6 -> 320.5 mm, vias 6 -> 4

Commit message: testing 5: DRC 9 errors/22 warnings -> 0 errors/1 warning
Routing:
- net +3.3V: track 104.6 -> 103.3 mm
- net GND: track 320.5 -> 319.7 mm
Changed lines of the file:
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@@
 		(tags "capacitor")
 		(property "Reference" "C5"
-			(at 0 -1.68 0)
+			(at 0 -3.355 0)
 			(layer "F.SilkS")
 			(effects
@@
 		(tags "CP Radial series Radial pin pitch 5.00mm diameter 10mm height 16mm Electrolytic Capacitor")
 		(property "Reference" "C4"
-			(at 2.5 -6.25 0)
+			(at 0.0004 6.675 0)
 			(layer "F.SilkS")
 			(effects
@@
 		(tags "capacitor")
 		(property "Reference" "C6"
-			(at 0 -1.16 0)
+			(at -1.995 3.845 0)
 			(layer "F.SilkS")
 			(effects
@@
 		(tags "CMS SOT")
 		(property "Reference" "U8"
-			(at 0 -4.5 0)
+			(at 0 -6.55 0)
 			(layer "F.SilkS")
 			(effects
@@
 		(tags "Resistor Axial_DIN0207 series Axial Horizontal pin pitch 7.62mm 0.25W = 1/4W length 6.3mm diameter 2.5mm")
 		(property "Reference" "R1"
-			(at 3.81 -2.37 0)
+			(at 3.81 3.3 0)
 			(layer "F.SilkS")
 			(effects
@@
 		(tags "capacitor")
 		(property "Reference" "C3"
-			(at 0 -1.16 0)
+			(at 0 3.2 0)
 			(layer "F.SilkS")
 			(effects
@@
 		(tags "capacitor")
 		(property "Reference" "C2"
-			(at 0 -1.68 0)
+			(at 2.8 3.2 0)
 			(layer "F.SilkS")
 			(effects
@@
 		(tags "capacitor")
 		(property "Reference" "C7"
-			(at 0 -1.68 0)
+			(at -2.785 -6.665 0)
 			(layer "F.SilkS")
 			(effects
@@
 		(fp_poly
 			(pts
-				(xy -9.2 -6.025) (xy -9.7 -6.025) (xy -9.2 -6.525)
+				(xy -9.2 -6.025) (xy -9.7 -6.025) (xy -9.2 -6.525) (xy -9.2 -6.025)
 			)
 			(stroke
@@
 				(clearance 0)
 			)
-			(min_thickness 0.25)
+			(min_thickness 0.254)
 			(keepout
 				(tracks not_allowed)
@@
 		(tags "capacitor")
 		(property "Reference" "C8"
-			(at 0 -1.16 0)
+			(at -2.695 -0.725 0)
 			(layer "F.SilkS")
 			(effects
@@
 	)
 	(segment
+		(start 152.8 87.7466)
+		(end 161.355 87.7466)
+		(width 0.25)
+		(layer "F.Cu")
+		(net "GND")
+	)
+	(segment
 		(start 115.075 79.725)
 		(end 115.075 77.755)
@@
 	)
 	(via
-		(at 181.15 88.5)
+		(at 115.075 81.5)
 		(size 0.8)
 		(drill 0.4)
@@
 	)
 	(via
-		(at 115.075 81.5)
-		(size 0.8)
-		(drill 0.4)
+		(at 152.8 87.7466)
+		(size 0.6)
+		(drill 0.3)
 		(layers "F.Cu" "B.Cu")
 		(net "GND")
@@
 	(segment
 		(start 115.075 92)
-		(end 171.1 92)
+		(end 152.8 92)
 		(width 0.25)
 		(layer "B.Cu")
@@
 	)
 	(segment
+		(start 152.8 92)
+		(end 152.8 87.7466)
+		(width 0.25)
+		(layer "B.Cu")
+		(net "GND")
+	)
+	(segment
+		(start 178.285 105.335)
+		(end 178.285 109.995)
+		(width 0.2)
+		(layer "B.Cu")
+		(net "GND")
+	)
+	(segment
 		(start 170.4 74.81)
 		(end 170.4 75.51)
@@
 	)
 	(segment
-		(start 165.602 69.06)
-		(end 165.867 69.06)
-		(width 0.2)
-		(layer "F.Cu")
-		(net "+3.3V")
-	)
-	(segment
 		(start 111.385 74.95)
 		(end 105.085 74.95)
@@
 		(width 0.2)
 		(layer "F.Cu")
-		(net "+3.3V")
-	)
-	(segment
-		(start 164.55 69.06)
-		(end 165.602 69.06)
-		(width 0.2)
-		(layer "F.Cu")
