File: testing 6/testing6.kicad_pcb (KiCad board)
At the start: 2 copper layers, 132 x 130 mm, 43 parts, among them J1 ESP32_GPIO, J2 Screw_Terminal_01x03, J3 Screw_Terminal_01x03, J4 Screw_Terminal_01x03, J5 Screw_Terminal_01x03, J6 USB_C_Receptacle_USB2.0_16P, K1 SRD-05VDC-SL-C, K2 SRD-05VDC-SL-C, K3 SRD-05VDC-SL-C, K4 SRD-05VDC-SL-C, SW1 RESET, SW2 BOOT, U1 ULN2003A, U2 PC817, U3 PC817, U4 PC817, U5 PC817, U6 ESP32-S3-WROOM-1, U7 HLK-PM01, U8 AMS1117-3.3, U9 CP2102N-Axx-xQFN20

Commit message: testing 6: user-routed USB section (7 tracks at 0.15mm, +3.3V island not yet joined)
Routing:
- net GND: track 319.7 -> 418.8 mm
- net /RXD0: track 0.00 -> 90.3 mm, vias 0 -> 2
- net /TXD0: track 0.00 -> 89.0 mm, vias 0 -> 2
- net /VBUS: track 0.00 -> 33.9 mm
- net /CC2: track 0.00 -> 23.1 mm, vias 0 -> 2
- net /CC1: track 0.00 -> 22.3 mm, vias 0 -> 2
- net /USB_D-: track 0.00 -> 18.7 mm
- net /USB_D+: track 0.00 -> 18.7 mm
- net +3.3V: track 103.3 -> 115.4 mm

Commit message: testing 6: route +3.3V to main rail, widen sub-minimum tracks, DRC 0 errors
Routing:
- net +3.3V: track 115.4 -> 197.0 mm, vias 2 -> 4
