File: testing 7/testing7.kicad_sch (KiCad schematic)
At the start: 43 parts, among them J1 ESP32_GPIO, J2 Screw_Terminal_01x03, J3 Screw_Terminal_01x03, J4 Screw_Terminal_01x03, J5 Screw_Terminal_01x03, J6 USB_C_Receptacle_USB2.0_16P, K1 SRD-05VDC-SL-C, K2 SRD-05VDC-SL-C, K3 SRD-05VDC-SL-C, K4 SRD-05VDC-SL-C, SW1 RESET, SW2 BOOT, U1 ULN2003A, U2 PC817, U3 PC817, U4 PC817, U5 PC817, U6 ESP32-S3-WROOM-1, U7 HLK-PM01, U8 AMS1117-3.3, U9 CP2102N-Axx-xQFN20

Commit message: testing 7: final combined schematic - 43 parts, 3 modules, ERC 0/0, 0 wires, A2 sheet
Other:
- note added: "1 POWER SUPPLY U7 HLK-PM01 -> U8 AMS1117-3.3 (+5V / +3.3V / GND)"
- note added: "2 RELAY MODULE U1 ULN2003A + 4 x PC817 opto + K1-K4 + D1-D4 flyback + J2-J5 loads + J1 GPIO"
- note added: "3 ESP32-S3 + SWITCHES U6 ESP32-S3-WROOM-1 + R5/R6 10k pull-ups + SW1 RESET / SW2 BOOT"
- note added: "4 USB PROGRAMMING J6 USB-C + U9 CP2102N + R7/R8 5.1k CC + C9/C10 100nF"
Changed lines of the file:
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@@
 	(generator "eeschema")
 	(generator_version "10.0")
-	(paper "A3")
+	(paper "A2")
 	(no_connect
 		(at 304.8 100.33)
@@
     (effects (font (size 1.5 1.5) (bold yes)) (justify left bottom))
   )
+  (text "1   POWER SUPPLY        U7 HLK-PM01  ->  U8 AMS1117-3.3   (+5V / +3.3V / GND)"
+    (at 44 62 0)
+    (effects (font (size 1.8 1.8) (bold yes)) (justify left bottom))
+  )
+  (text "2   RELAY MODULE        U1 ULN2003A  +  4 x PC817 opto  +  K1-K4  +  D1-D4 flyback  +  J2-J5 loads  +  J1 GPIO"
+    (at 44 38 0)
+    (effects (font (size 1.8 1.8) (bold yes)) (justify left bottom))
+  )
+  (text "3   ESP32-S3 + SWITCHES        U6 ESP32-S3-WROOM-1  +  R5/R6 10k pull-ups  +  SW1 RESET / SW2 BOOT"
+    (at 272 34 0)
+    (effects (font (size 1.8 1.8) (bold yes)) (justify left bottom))
+  )
+  (text "4   USB PROGRAMMING        J6 USB-C  +  U9 CP2102N  +  R7/R8 5.1k CC  +  C9/C10 100nF"
+    (at 240 228 0)
+    (effects (font (size 1.8 1.8) (bold yes)) (justify left bottom))
+  )
 	(symbol
